File: _pcb/RoombaESP.sch (KiCad schematic (older format))
At the start: 11 parts, among them J1 LDR, J2 LCD, J3 ROOMBA SER, J4 SW/LED, U1 WeMos_D1_mini, U2 HW-613

Commit message: Added RoombaESP PCB v2.0
Parts:
- removed U2: HW-613, HW-613:HW-613, symbol HW-613:HW-613
- added U2: DD4012SA, Converter_DCDC_Mod:DD4012SA, symbol Converter_DCDC_Mod:DD4012SA
- J1: footprint Connector_PinHeader_2.54mm:PinHeader_1x02_P2.54mm_Horizontal -> Connector_JST:JST_PH_S2B-PH-K_1x02_P2.00mm_Horizontal
- J2: renamed from J4; footprint Connector_PinHeader_2.54mm:PinHeader_1x03_P2.54mm_Horizontal -> Connector_JST:JST_PH_S3B-PH-K_1x03_P2.00mm_Horizontal
- J3: renamed from J2; footprint Connector_PinHeader_2.54mm:PinHeader_1x04_P2.54mm_Horizontal -> Connector_JST:JST_PH_S4B-PH-K_1x04_P2.00mm_Horizontal
- J4: renamed from J3; footprint Connector_PinHeader_2.54mm:PinHeader_1x05_P2.54mm_Horizontal -> Connector_JST:JST_PH_S5B-PH-K_1x05_P2.00mm_Horizontal
- R1: value 20K -> 10K
- R2: value 10K -> 6.8K
Connections:
- net labels added: LCD_SCL
- net labels removed: LCD_SDL
- no-connect marks 7 -> 6
Other:
- moved on the sheet: J2, J4
Changed lines of the file:
@@
 $EndComp
 $Comp
-L Connector:Conn_01x04_Male J2
+L Connector:Conn_01x04_Male J3
 U 1 1 5FE99303
-P 5950 1800
-F 0 "J2" H 5922 1774 50  0000 R CNN
-F 1 "LCD" H 5922 1683 50  0000 R CNN
-F 2 "Connector_PinHeader_2.54mm:PinHeader_1x04_P2.54mm_Horizontal" H 5950 1800 50  0001 C CNN
-F 3 "~" H 5950 1800 50  0001 C CNN
-	1    5950 1800
-	-1   0    0    -1
-$EndComp
-$Comp
-L Connector:Conn_01x03_Male J4
+P 5950 1900
+F 0 "J3" H 5922 1874 50  0000 R CNN
+F 1 "LCD" H 5922 1783 50  0000 R CNN
+F 2 "Connector_JST:JST_PH_S4B-PH-K_1x04_P2.00mm_Horizontal" H 5950 1900 50  0001 C CNN
+F 3 "~" H 5950 1900 50  0001 C CNN
+	1    5950 1900
+	-1   0    0    1
+$EndComp
+$Comp
+L Connector:Conn_01x03_Male J2
 U 1 1 5FE9A213
-P 5950 2900
-F 0 "J4" H 5922 2924 50  0000 R CNN
-F 1 "SW/LED" H 5922 2833 50  0000 R CNN
-F 2 "Connector_PinHeader_2.54mm:PinHeader_1x03_P2.54mm_Horizontal" H 5950 2900 50  0001 C CNN
-F 3 "~" H 5950 2900 50  0001 C CNN
-	1    5950 2900
-	-1   0    0    -1
-$EndComp
-$Comp
-L HW-613:HW-613 U2
-U 1 1 5FE9FC12
-P 3250 1300
-F 0 "U2" H 3400 1600 50  0000 L CNN
-F 1 "HW-613" H 2950 1600 50  0000 L CNN
-F 2 "HW-613:HW-613" H 3250 1700 50  0000 C CNN
-F 3 "" H 3300 1650 50  0001 C CNN
-	1    3250 1300
-	1    0    0    -1
-$EndComp
-$Comp
-L power:GND #PWR0101
-U 1 1 5FEA17E1
-P 3650 1250
-F 0 "#PWR0101" H 3650 1000 50  0001 C CNN
-F 1 "GND" V 3650 1000 50  0000 C CNN
-F 2 "" H 3650 1250 50  0001 C CNN
-F 3 "" H 3650 1250 50  0001 C CNN
-	1    3650 1250
-	0    -1   -1   0
+P 5950 2300
+F 0 "J2" H 5922 2324 50  0000 R CNN
+F 1 "SW/LED" H 5922 2233 50  0000 R CNN
+F 2 "Connector_JST:JST_PH_S3B-PH-K_1x03_P2.00mm_Horizontal" H 5950 2300 50  0001 C CNN
+F 3 "~" H 5950 2300 50  0001 C CNN
+	1    5950 2300
+	-1   0    0    1
 $EndComp
 $Comp
@@
 	1    0    0    -1
 $EndComp
-Text GLabel 3650 1350 2    50   Input ~ 0
-RMB_PWR
-NoConn ~ 3650 1450
-$Comp
-L Connector:Conn_01x05_Male J3
+$Comp
+L Connector:Conn_01x05_Male J4
 U 1 1 5FEA7263
-P 5950 2400
-F 0 "J3" H 5922 2424 50  0000 R CNN
-F 1 "ROOMBA SER" H 5922 2333 50  0000 R CNN
-F 2 "Connector_PinHeader_2.54mm:PinHeader_1x05_P2.54mm_Horizontal" H 5950 2400 50  0001 C CNN
-F 3 "~" H 5950 2400 50  0001 C CNN
-	1    5950 2400
-	-1   0    0    -1
-$EndComp
-Text GLabel 5750 2200 0    50   Input ~ 0
+P 6000 2850
+F 0 "J4" H 5972 2874 50  0000 R CNN
+F 1 "ROOMBA SER" H 5972 2783 50  0000 R CNN
+F 2 "Connector_JST:JST_PH_S5B-PH-K_1x05_P2.00mm_Horizontal" H 6000 2850 50  0001 C CNN
+F 3 "~" H 6000 2850 50  0001 C CNN
+	1    6000 2850
+	-1   0    0    1
+$EndComp
+Text GLabel 5800 2650 0    50   Input ~ 0
 RMB_BRC
-Text GLabel 5750 2400 0    50   Input ~ 0
+Text GLabel 5800 2850 0    50   Input ~ 0
+RMB_RXD
+Text GLabel 5800 2950 0    50   Input ~ 0
 RMB_TXD
-Text GLabel 5750 2500 0    50   Input ~ 0
-RMB_RXD
-Text GLabel 5750 2600 0    50   Input ~ 0
+Text GLabel 5800 3050 0    50   Input ~ 0
 RMB_PWR
 $Comp
 L power:GND #PWR0106
 U 1 1 5FEAC797
-P 5750 3000
-F 0 "#PWR0106" H 5750 2750 50  0001 C CNN
-F 1 "GND" V 5755 2872 50  0000 R CNN
-F 2 "" H 5750 3000 50  0001 C CNN
-F 3 "" H 5750 3000 50  0001 C CNN
-	1    5750 3000
-	0    1    1    0
-$EndComp
-Text GLabel 5750 2900 0    50   Input ~ 0
+P 5750 2400
+F 0 "#PWR0106" H 5750 2150 50  0001 C CNN
+F 1 "GND" V 5755 2272 50  0000 R CNN
+F 2 "" H 5750 2400 50  0001 C CNN
+F 3 "" H 5750 2400 50  0001 C CNN
+	1    5750 2400
+	0    1    1    0
+$EndComp
+Text GLabel 5750 2300 0    50   Input ~ 0
 SW_BTN
-Text GLabel 5750 2800 0    50   Input ~ 0
+Text GLabel 5750 2200 0    50   Input ~ 0
 SW_LED
 $Comp
@@
 $EndComp
 Text GLabel 5750 1900 0    50   Input ~ 0
-LCD_SDL
+LCD_SCL
 Text GLabel 5750 2000 0    50   Input ~ 0
 LCD_SDA
@@
 P 3800 3350
 F 0 "R1" V 3593 3350 50  0000 C CNN
-F 1 "20K" V 3684 3350 50  0000 C CNN
+F 1 "10K" V 3684 3350 50  0000 C CNN
 F 2 "Resistor_SMD:R_0805_2012Metric_Pad1.20x1.40mm_HandSolder" V 3730 3350 50  0001 C CNN
 F 3 "~" H 3800 3350 50  0001 C CNN
@@
 P 4100 3350
 F 0 "R2" V 3893 3350 50  0000 C CNN
-F 1 "10K" V 3984 3350 50  0000 C CNN
+F 1 "6.8K" V 3984 3350 50  0000 C CNN
 F 2 "Resistor_SMD:R_0805_2012Metric_Pad1.20x1.40mm_HandSolder" V 4030 3350 50  0001 C CNN
 F 3 "~" H 4100 3350 50  0001 C CNN
@@
 L Connector:Conn_01x02_Male J1
 U 1 1 5FED6D2E
-P 5950 1500
-F 0 "J1" H 5922 1382 50  0000 R CNN
-F 1 "LDR" H 5922 1473 50  0000 R CNN
-F 2 "Connector_PinHeader_2.54mm:PinHeader_1x02_P2.54mm_Horizontal" H 5950 1500 50  0001 C CNN
-F 3 "~" H 5950 1500 50  0001 C CNN
-	1    5950 1500
-	-1   0    0    1
+P 5950 1400
+F 0 "J1" H 5900 1400 50  0000 R CNN
+F 1 "LDR" H 5900 1300 50  0000 R CNN
+F 2 "Connector_JST:JST_PH_S2B-PH-K_1x02_P2.00mm_Horizontal" H 5950 1400 50  0001 C CNN
+F 3 "~" H 5950 1400 50  0001 C CNN
+	1    5950 1400
+	-1   0    0    -1
 $EndComp
 $Comp
@@
 LCD_SDA
 Text GLabel 1950 1950 2    50   Input ~ 0
-LCD_SDL
+LCD_SCL
 NoConn ~ 1950 1350
 NoConn ~ 1950 1750
@@
 $EndComp
 $Comp
-L power:+3.3V #PWR0104
-U 1 1 5FF25108
-P 3650 1150
-F 0 "#PWR0104" H 3650 1000 50  0001 C CNN
-F 1 "+3.3V" V 3650 1300 50  0000 L CNN
-F 2 "" H 3650 1150 50  0001 C CNN
-F 3 "" H 3650 1150 50  0001 C CNN
-	1    3650 1150
-	0    1    1    0
-$EndComp
-$Comp
 L power:GND #PWR0109
 U 1 1 5FF262A9
@@
 L power:GND #PWR0105
 U 1 1 5FEBC77D
-P 5750 2300
-F 0 "#PWR0105" H 5750 2050 50  0001 C CNN
-F 1 "GND" V 5755 2172 50  0000 R CNN
-F 2 "" H 5750 2300 50  0001 C CNN
-F 3 "" H 5750 2300 50  0001 C CNN
-	1    5750 2300
-	0    1    1    0
+P 5800 2750
+F 0 "#PWR0105" H 5800 2500 50  0001 C CNN
+F 1 "GND" V 5805 2622 50  0000 R CNN
+F 2 "" H 5800 2750 50  0001 C CNN
+F 3 "" H 5800 2750 50  0001 C CNN
+	1    5800 2750
+	0    1    1    0
+$EndComp
+Text GLabel 3900 1300 2    50   Input ~ 0
+RMB_PWR
+$Comp
+L power:GND #PWR0101
+U 1 1 600B3CE3
+P 3900 1400
+F 0 "#PWR0101" H 3900 1150 50  0001 C CNN
+F 1 "GND" V 3905 1272 50  0000 R CNN
+F 2 "" H 3900 1400 50  0001 C CNN
+F 3 "" H 3900 1400 50  0001 C CNN
+	1    3900 1400
+	0    -1   -1   0
+$EndComp
+$Comp
+L power:+3.3V #PWR0104
+U 1 1 600B4C35
+P 3900 1500
+F 0 "#PWR0104" H 3900 1350 50  0001 C CNN
+F 1 "+3.3V" V 3915 1628 50  0000 L CNN
+F 2 "" H 3900 1500 50  0001 C CNN
+F 3 "" H 3900 1500 50  0001 C CNN
+	1    3900 1500
+	0    1    1    0
+$EndComp
+$Comp
+L Converter_DCDC_Mod:DD4012SA U2
+U 1 1 600BABF8
+P 3650 1350
+F 0 "U2" H 3708 1715 50  0000 C CNN
+F 1 "DD4012SA" H 3708 1624 50  0000 C CNN
+F 2 "Converter_DCDC_Mod:DD4012SA" H 3708 1533 50  0000 C CNN
+F 3 "" H 3650 1500 50  0001 C CNN
+	1    3650 1350
+	1    0    0    -1
 $EndComp
 $EndSCHEMATC
